Commit message: added cylindrical endeff to kuka arm

File: models/arms/ball_arm.urdf (robot description, URDF)
Before this commit: robot robot_gripper, 2 links, 1 joints
Links:
- link gripper_ball: geometry collision sphere radius=0.04; visual sphere radius=0.04

File: models/objects/block1.urdf (robot description, URDF)
Before this commit: robot block1, 1 links, 0 joints
Links:
- link block1_base_link: mass 0.02 -> 0.2; geometry collision box size=0.4 0.15 0.05; visual box size=0.4 0.15 0.05

File: models/objects/block2.urdf (robot description, URDF)
Before this commit: robot block2, 1 links, 0 joints
Links:
- link block2_base_link: mass 0.02 -> 0.2; geometry collision box size=0.15 0.45 0.15; visual box size=0.15 0.45 0.15

Commit message: generate qs trajs for floating arm env

File: models/arms/ball_arm.urdf (robot description, URDF)
Before this commit: robot robot_gripper, 2 links, 1 joints
Links:
- link gripper_pole: mass 0.5 -> 1.0

File: models/objects/block1.urdf (robot description, URDF)
Before this commit: robot block1, 1 links, 0 joints
Links:
- link block1_base_link: mass 0.2 -> 0.5

File: models/objects/block2.urdf (robot description, URDF)
Before this commit: robot block2, 1 links, 0 joints
Links:
- link block2_base_link: mass 0.2 -> 0.5; geometry collision box size=0.15 0.40 0.15; visual box size=0.15 0.40 0.15
